File: avrisp.kicad_pcb (KiCad board)
At the start: 2 copper layers, 25 parts, among them J3 USB_A, J4 CONN_02X05, U1 ATMEGA8-16PU, Y1 12MHz

Commit message: Update PCB
Parts:
- moved D3 103.2 mm to (56.0, 77.0)
- moved D4 95.2 mm to (64.0, 76.0)
- moved R10 74.3 mm to (65.2, 103.0), turned to 180 degrees
- moved JP3 56.4 mm to (108.0, 109.0)
- moved J4 55.7 mm to (123.5, 94.2)
- moved C4 55.7 mm to (96.0, 90.0), turned to 270 degrees
- moved C3 51.1 mm to (101.0, 91.2), turned to 270 degrees
- moved JP1 41.6 mm to (99.0, 109.0)
- moved R6 25.2 mm to (105.2, 104.0), turned to 180 degrees
- moved Y1 6.57 mm to (73.1, 85.0), turned to 0 degrees
- moved JP2 3.68 mm to (77.5, 107.0)
Routing:
- net +5V: track 0.00 -> 86.0 mm
- net GND: track 34.6 -> 87.8 mm
- net Net-(J4-Pad1): track 0.00 -> 29.6 mm
- net Net-(J4-Pad5): track 0.00 -> 23.3 mm
- net Net-(J4-Pad2): track 0.00 -> 22.3 mm
- net Net-(D4-Pad3): track 16.2 -> 38.3 mm
- net Net-(D3-Pad3): track 53.7 -> 73.5 mm
- net Net-(R6-Pad2): track 0.00 -> 19.5 mm
- net Net-(JP2-Pad1): track 0.00 -> 16.1 mm
- net Net-(JP1-Pad1): track 0.00 -> 13.6 mm
- net Net-(C1-Pad1): track 20.9 -> 17.3 mm
- net Net-(C2-Pad1): track 14.5 -> 11.2 mm
- net Net-(J4-Pad9): track 0.00 -> 0.54 mm

Commit message: Finish PCB
Parts:
- moved JP3 6.08 mm to (111.5, 104.0)
Routing:
- net Net-(J4-Pad5): track 23.3 -> 128.4 mm
- net Net-(J4-Pad6): track 0.00 -> 63.6 mm
- net Net-(J4-Pad9): track 0.54 -> 34.2 mm
- net Net-(J4-Pad4): track 0.00 -> 33.2 mm
- net Net-(J4-Pad7): track 0.00 -> 18.5 mm
- net Net-(J4-Pad2): track 22.3 -> 16.8 mm
- net +5V: track 86.0 -> 81.2 mm
- net GND: track 87.8 -> 90.9 mm
- net Net-(D4-Pad3): track 38.3 -> 39.2 mm
- added copper zone on B.Cu, net GND
- added copper zone on F.Cu, net GND
Other:
- net class Default: trace_width 0.5 -> 0.6; via_drill 0.9 -> 0.5
- rule via_min_size: 1 -> 0.5

Commit message: Make one side version
Parts:
- moved C1 68.0 mm to (35.2, 23.0)
- moved C2 68.0 mm to (40.8, 23.0)
- moved C3 68.0 mm to (64.0, 34.2)
- moved C4 68.0 mm to (59.0, 33.0)
- moved D1 68.0 mm to (59.0, 39.0)
- moved D2 68.0 mm to (59.0, 42.0)
- moved D3 68.0 mm to (19.0, 20.1)
- moved D4 68.0 mm to (27.0, 19.0)
- moved J3 68.0 mm to (28.0, 35.5)
- moved J4 68.0 mm to (86.5, 37.2)
- moved JP1 68.0 mm to (62.0, 52.0)
- moved JP2 68.0 mm to (40.5, 50.0)
- moved JP3 68.0 mm to (74.5, 47.0)
- moved R1 68.0 mm to (31.8, 41.0)
- moved R10 68.0 mm to (28.2, 46.0)
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Connections:
- JP2 pad 2: Net-(J4-Pad5) -> Net-(J4-Pad9)
- R3 pad 1: Net-(J4-Pad5) -> Net-(J4-Pad9)
- R4 pad 1: Net-(J4-Pad1) -> Net-(J4-Pad7)
- R5 pad 1: Net-(J4-Pad7) -> Net-(J4-Pad1)
- U1 pad 18: Net-(J4-Pad9) -> Net-(J4-Pad5)
Routing:
- net Net-(J4-Pad5): track 128.4 -> 35.8 mm
- net Net-(J4-Pad9): track 34.2 -> 108.0 mm
- net +5V: track 81.2 -> 111.3 mm
- net Net-(J4-Pad1): track 29.6 -> 25.1 mm
- net Net-(J4-Pad7): track 18.5 -> 21.4 mm
- net Net-(R9-Pad1): track 33.8 -> 35.1 mm
- net Net-(JP1-Pad1): track 13.6 -> 14.6 mm
- removed copper zone on B.Cu, net GND
Other:
- net class 1 added: clearance 0.7, trace_width 0.6, via_dia 1.2, via_drill 0.5
