File: avrisp.sch (KiCad schematic (older format))
At the start: 25 parts, among them J3 USB_A, J4 CONN_02X05, U1 ATMEGA8-16PU, Y1 12MHz

Commit message: Make few fixes
Connections:
- net +5V: now also U1.7 (VCC)
Changed lines of the file:
@@
 U 1 1 5921E579
 P 4650 4200
-F 0 "U1" H 4700 5778 50  0000 C CNN
-F 1 "ATMEGA8-16PU" H 4700 5687 50  0000 C CNN
+F 0 "U1" H 3950 5550 50  0000 C CNN
+F 1 "ATMEGA8-16PU" H 5200 5550 50  0000 C CNN
 F 2 "DIL28" H 4650 4200 50  0001 C CIN
 F 3 "" H 4650 4200 50  0001 C CNN
@@
 $EndComp
 $Comp
-L +5V #PWR7
+L +5V #PWR01
 U 1 1 5921E649
 P 5900 2050
-F 0 "#PWR7" H 5900 1900 50  0001 C CNN
+F 0 "#PWR01" H 5900 1900 50  0001 C CNN
 F 1 "+5V" H 5915 2223 50  0000 C CNN
 F 2 "" H 5900 2050 50  0001 C CNN
@@
 $EndComp
 $Comp
-L +5V #PWR8
+L +5V #PWR02
 U 1 1 5921E662
 P 6300 2050
-F 0 "#PWR8" H 6300 1900 50  0001 C CNN
+F 0 "#PWR02" H 6300 1900 50  0001 C CNN
 F 1 "+5V" H 6315 2223 50  0000 C CNN
 F 2 "" H 6300 2050 50  0001 C CNN
@@
 $EndComp
 $Comp
-L +5V #PWR4
+L +5V #PWR03
 U 1 1 5921E7C3
 P 3500 2600
-F 0 "#PWR4" H 3500 2450 50  0001 C CNN
+F 0 "#PWR03" H 3500 2450 50  0001 C CNN
 F 1 "+5V" H 3515 2773 50  0000 C CNN
 F 2 "" H 3500 2600 50  0001 C CNN
@@
 $EndComp
 $Comp
-L +5V #PWR3
+L +5V #PWR04
 U 1 1 5921E7DA
 P 3200 2600
-F 0 "#PWR3" H 3200 2450 50  0001 C CNN
+F 0 "#PWR04" H 3200 2450 50  0001 C CNN
 F 1 "+5V" H 3215 2773 50  0000 C CNN
 F 2 "" H 3200 2600 50  0001 C CNN
@@
 $EndComp
 $Comp
-L GND #PWR5
+L GND #PWR05
 U 1 1 5921E82A
 P 3600 4150
-F 0 "#PWR5" H 3600 3900 50  0001 C CNN
+F 0 "#PWR05" H 3600 3900 50  0001 C CNN
 F 1 "GND" H 3605 3977 50  0000 C CNN
 F 2 "" H 3600 4150 50  0001 C CNN
@@
 	3600 3500 3600 4150
 $Comp
-L GND #PWR6
+L GND #PWR06
 U 1 1 5921E86E
 P 4650 5800
-F 0 "#PWR6" H 4650 5550 50  0001 C CNN
+F 0 "#PWR06" H 4650 5550 50  0001 C CNN
 F 1 "GND" H 4655 5627 50  0000 C CNN
 F 2 "" H 4650 5800 50  0001 C CNN
@@
 NoConn ~ 3750 3400
 $Comp
-L +5V #PWR15
+L +5V #PWR07
 U 1 1 5921E8E5
 P 8850 1350
-F 0 "#PWR15" H 8850 1200 50  0001 C CNN
+F 0 "#PWR07" H 8850 1200 50  0001 C CNN
 F 1 "+5V" H 8865 1523 50  0000 C CNN
 F 2 "" H 8850 1350 50  0001 C CNN
@@
 $EndComp
 $Comp
-L +5V #PWR17
+L +5V #PWR08
 U 1 1 5921E8F8
 P 9350 1350
-F 0 "#PWR17" H 9350 1200 50  0001 C CNN
+F 0 "#PWR08" H 9350 1200 50  0001 C CNN
 F 1 "+5V" H 9365 1523 50  0000 C CNN
 F 2 "" H 9350 1350 50  0001 C CNN
@@
 $EndComp
 $Comp
-L GND #PWR16
+L GND #PWR09
 U 1 1 5921EA04
 P 8850 1650
-F 0 "#PWR16" H 8850 1400 50  0001 C CNN
+F 0 "#PWR09" H 8850 1400 50  0001 C CNN
 F 1 "GND" H 8855 1477 50  0000 C CNN
 F 2 "" H 8850 1650 50  0001 C CNN
@@
 $EndComp
 $Comp
-L GND #PWR18
+L GND #PWR010
 U 1 1 5921EA1B
 P 9350 1650
-F 0 "#PWR18" H 9350 1400 50  0001 C CNN
+F 0 "#PWR010" H 9350 1400 50  0001 C CNN
 F 1 "GND" H 9355 1477 50  0000 C CNN
 F 2 "" H 9350 1650 50  0001 C CNN
@@
 Connection ~ 2400 4000
 $Comp
-L GND #PWR2
+L GND #PWR011
 U 1 1 5921EE36
 P 2950 4600
-F 0 "#PWR2" H 2950 4350 50  0001 C CNN
+F 0 "#PWR011" H 2950 4350 50  0001 C CNN
 F 1 "GND" H 2955 4427 50  0000 C CNN
 F 2 "" H 2950 4600 50  0001 C CNN
@@
 $EndComp
 $Comp
-L GND #PWR1
+L GND #PWR012
 U 1 1 5921EE53
 P 2400 4600
-F 0 "#PWR1" H 2400 4350 50  0001 C CNN
+F 0 "#PWR012" H 2400 4350 50  0001 C CNN
 F 1 "GND" H 2405 4427 50  0000 C CNN
 F 2 "" H 2400 4600 50  0001 C CNN
@@
 	6850 3200 6700 3200
 $Comp
-L +5V #PWR14
+L +5V #PWR013
 U 1 1 59220993
 P 8350 2750
-F 0 "#PWR14" H 8350 2600 50  0001 C CNN
+F 0 "#PWR013" H 8350 2600 50  0001 C CNN
 F 1 "+5V" H 8365 2923 50  0000 C CNN
 F 2 "" H 8350 2750 50  0001 C CNN
@@
 $EndComp
 $Comp
-L GND #PWR19
+L GND #PWR014
 U 1 1 592209F9
 P 9350 2850
-F 0 "#PWR19" H 9350 2600 50  0001 C CNN
+F 0 "#PWR014" H 9350 2600 50  0001 C CNN
 F 1 "GND" H 9355 2677 50  0000 C CNN
 F 2 "" H 9350 2850 50  0001 C CNN
@@
 $EndComp
 $Comp
-L GND #PWR13
+L GND #PWR015
 U 1 1 59220F59
 P 8000 5000
-F 0 "#PWR13" H 8000 4750 50  0001 C CNN
+F 0 "#PWR015" H 8000 4750 50  0001 C CNN
 F 1 "GND" H 8005 4827 50  0000 C CNN
 F 2 "" H 8000 5000 50  0001 C CNN
@@
 Connection ~ 8000 4800
 $Comp
-L +5V #PWR20
+L +5V #PWR016
 U 1 1 592212AC
 P 10000 3800
-F 0 "#PWR20" H 10000 3650 50  0001 C CNN
+F 0 "#PWR016" H 10000 3650 50  0001 C CNN
 F 1 "+5V" H 10015 3973 50  0000 C CNN
 F 2 "" H 10000 3800 50  0001 C CNN
@@
 $EndComp
 $Comp
-L +5V #PWR10
+L +5V #PWR017
 U 1 1 59223BEE
 P 6900 2650
-F 0 "#PWR10" H 6900 2500 50  0001 C CNN
+F 0 "#PWR017" H 6900 2500 50  0001 C CNN
 F 1 "+5V" H 6915 2823 50  0000 C CNN
 F 2 "" H 6900 2650 50  0001 C CNN
@@
 $EndComp
 $Comp
-L GND #PWR9
+L GND #PWR018
 U 1 1 592245AF
 P 6300 5450
-F 0 "#PWR9" H 6300 5200 50  0001 C CNN
+F 0 "#PWR018" H 6300 5200 50  0001 C CNN
 F 1 "GND" H 6305 5277 50  0000 C CNN
 F 2 "" H 6300 5450 50  0001 C CNN
@@
 Connection ~ 7700 3300
 $Comp
-L GND #PWR11
+L GND #PWR019
 U 1 1 59225578
 P 7300 3750
-F 0 "#PWR11" H 7300 3500 50  0001 C CNN
+F 0 "#PWR019" H 7300 3500 50  0001 C CNN
 F 1 "GND" H 7305 3577 50  0000 C CNN
 F 2 "" H 7300 3750 50  0001 C CNN
@@
 $EndComp
 $Comp
-L GND #PWR12
+L GND #PWR020
 U 1 1 592255B5
 P 7700 3750
-F 0 "#PWR12" H 7700 3500 50  0001 C CNN
+F 0 "#PWR020" H 7700 3500 50  0001 C CNN
 F 1 "GND" H 7705 3577 50  0000 C CNN
 F 2 "" H 7700 3750 50  0001 C CNN
@@
 	1    0    0    -1
 $EndComp
+$Comp
+L PWR_FLAG #FLG021
+U 1 1 5922614D
+P 3250 3600
+F 0 "#FLG021" H 3250 3675 50  0001 C CNN
+F 1 "PWR_FLAG" H 3250 3774 50  0000 C CNN
+F 2 "" H 3250 3600 50  0001 C CNN
+F 3 "" H 3250 3600 50  0001 C CNN
+	1    3250 3600
+	1    0    0    -1
+$EndComp
+Wire Wire Line
+	3250 3600 3250 3700
+Wire Wire Line
+	3250 3700 3600 3700
+Connection ~ 3600 3700
+$Comp
+L PWR_FLAG #FLG022
+U 1 1 59226374
+P 2850 2750
+F 0 "#FLG022" H 2850 2825 50  0001 C CNN
+F 1 "PWR_FLAG" H 2850 2924 50  0000 C CNN
+F 2 "" H 2850 2750 50  0001 C CNN
+F 3 "" H 2850 2750 50  0001 C CNN
+	1    2850 2750
+	1    0    0    -1
+$EndComp
+Wire Wire Line
+	2850 2750 2850 2850
+Wire Wire Line
+	2850 2850 3200 2850
+Connection ~ 3200 2850
+$Comp
+L +5V #PWR023
+U 1 1 59229303
+P 4650 2350
+F 0 "#PWR023" H 4650 2200 50  0001 C CNN
+F 1 "+5V" H 4665 2523 50  0000 C CNN
+F 2 "" H 4650 2350 50  0001 C CNN
+F 3 "" H 4650 2350 50  0001 C CNN
+	1    4650 2350
+	1    0    0    -1
+$EndComp
+Wire Wire Line
+	4650 2800 4650 2350
 $EndSCHEMATC

Commit message: Modify PCB
Parts:
- removed D3, D4: 3V6, symbol D_Zener
- added D3, D4: 3V6, symbol D_Zener_SOT23
- C1, C2, C3: footprint (none) -> Capacitors_SMD:C_0805_HandSoldering
- C4: footprint (none) -> Capacitors_THT:CP_Radial_D4.0mm_P2.00mm
- D1, D2: footprint (none) -> LEDs:LED_1206
- J3: footprint (none) -> Connectors:USB_A
- J4: footprint (none) -> Connectors:IDC_Header_Straight_10pins
- JP1, JP2, JP3: footprint (none) -> Connectors_Molex:Molex_KK-6410-02_02x2.54mm_Straight
- R1, R10, R2, R3, R4, R5, R6, R7, R8, R9: footprint (none) -> Resistors_THT:R_Axial_DIN0207_L6.3mm_D2.5mm_P10.16mm_Horizontal
- U1: footprint DIL28 -> Housings_DIP:DIP-28_W7.62mm
- Y1: footprint (none) -> Crystals:Crystal_HC50_Vertical
Connections:
- net GND: now also D3.1 (A), D4.1 (A)
- net at J3.2 (D-), R10.2, R8.2: now also D4.3 (K)
- net at J3.3 (D+), R9.2: now also D3.3 (K)

Commit message: Update PCB
Parts:
- D3, D4: footprint (none) -> TO_SOT_Packages_SMD:SOT-23
Changed lines of the file:
@@
 $EndComp
 $Comp
-L +5V #PWR8
+L +5V #PWR01
 U 1 1 5921E649
 P 5900 2050
-F 0 "#PWR8" H 5900 1900 50  0001 C CNN
+F 0 "#PWR01" H 5900 1900 50  0001 C CNN
 F 1 "+5V" H 5915 2223 50  0000 C CNN
 F 2 "" H 5900 2050 50  0001 C CNN
@@
 $EndComp
 $Comp
-L +5V #PWR9
+L +5V #PWR02
 U 1 1 5921E662
 P 6300 2050
-F 0 "#PWR9" H 6300 1900 50  0001 C CNN
+F 0 "#PWR02" H 6300 1900 50  0001 C CNN
 F 1 "+5V" H 6315 2223 50  0000 C CNN
 F 2 "" H 6300 2050 50  0001 C CNN
@@
 $EndComp
 $Comp
-L +5V #PWR4
+L +5V #PWR03
 U 1 1 5921E7C3
 P 3500 2600
-F 0 "#PWR4" H 3500 2450 50  0001 C CNN
+F 0 "#PWR03" H 3500 2450 50  0001 C CNN
 F 1 "+5V" H 3515 2773 50  0000 C CNN
 F 2 "" H 3500 2600 50  0001 C CNN
@@
 $EndComp
 $Comp
-L +5V #PWR3
+L +5V #PWR04
 U 1 1 5921E7DA
 P 3200 2600
-F 0 "#PWR3" H 3200 2450 50  0001 C CNN
+F 0 "#PWR04" H 3200 2450 50  0001 C CNN
 F 1 "+5V" H 3215 2773 50  0000 C CNN
 F 2 "" H 3200 2600 50  0001 C CNN
@@
 $EndComp
 $Comp
-L GND #PWR5
+L GND #PWR05
 U 1 1 5921E82A
 P 3600 4150
-F 0 "#PWR5" H 3600 3900 50  0001 C CNN
+F 0 "#PWR05" H 3600 3900 50  0001 C CNN
 F 1 "GND" H 3605 3977 50  0000 C CNN
 F 2 "" H 3600 4150 50  0001 C CNN
@@
 	3600 3500 3600 4150
 $Comp
-L GND #PWR7
+L GND #PWR06
 U 1 1 5921E86E
 P 4650 5800
-F 0 "#PWR7" H 4650 5550 50  0001 C CNN
+F 0 "#PWR06" H 4650 5550 50  0001 C CNN
 F 1 "GND" H 4655 5627 50  0000 C CNN
 F 2 "" H 4650 5800 50  0001 C CNN
@@
 NoConn ~ 3750 3400
 $Comp
-L +5V #PWR16
+L +5V #PWR07
 U 1 1 5921E8E5
 P 8850 1350
-F 0 "#PWR16" H 8850 1200 50  0001 C CNN
+F 0 "#PWR07" H 8850 1200 50  0001 C CNN
 F 1 "+5V" H 8865 1523 50  0000 C CNN
 F 2 "" H 8850 1350 50  0001 C CNN
@@
 $EndComp
 $Comp
-L +5V #PWR18
+L +5V #PWR08
 U 1 1 5921E8F8
 P 9350 1350
-F 0 "#PWR18" H 9350 1200 50  0001 C CNN
+F 0 "#PWR08" H 9350 1200 50  0001 C CNN
 F 1 "+5V" H 9365 1523 50  0000 C CNN
 F 2 "" H 9350 1350 50  0001 C CNN
@@
 $EndComp
 $Comp
-L GND #PWR17
+L GND #PWR09
 U 1 1 5921EA04
 P 8850 1650
-F 0 "#PWR17" H 8850 1400 50  0001 C CNN
+F 0 "#PWR09" H 8850 1400 50  0001 C CNN
 F 1 "GND" H 8855 1477 50  0000 C CNN
 F 2 "" H 8850 1650 50  0001 C CNN
@@
 $EndComp
 $Comp
-L GND #PWR19
+L GND #PWR010
 U 1 1 5921EA1B
 P 9350 1650
-F 0 "#PWR19" H 9350 1400 50  0001 C CNN
+F 0 "#PWR010" H 9350 1400 50  0001 C CNN
 F 1 "GND" H 9355 1477 50  0000 C CNN
 F 2 "" H 9350 1650 50  0001 C CNN
@@
 Connection ~ 2400 4000
 $Comp
-L GND #PWR2
+L GND #PWR011
 U 1 1 5921EE36
 P 2950 4600
-F 0 "#PWR2" H 2950 4350 50  0001 C CNN
+F 0 "#PWR011" H 2950 4350 50  0001 C CNN
 F 1 "GND" H 2955 4427 50  0000 C CNN
 F 2 "" H 2950 4600 50  0001 C CNN
@@
 $EndComp
 $Comp
-L GND #PWR1
+L GND #PWR012
 U 1 1 5921EE53
 P 2400 4600
-F 0 "#PWR1" H 2400 4350 50  0001 C CNN
+F 0 "#PWR012" H 2400 4350 50  0001 C CNN
 F 1 "GND" H 2405 4427 50  0000 C CNN
 F 2 "" H 2400 4600 50  0001 C CNN
@@
 	6850 3200 6700 3200
 $Comp
-L +5V #PWR15
+L +5V #PWR013
 U 1 1 59220993
 P 8350 2750
-F 0 "#PWR15" H 8350 2600 50  0001 C CNN
+F 0 "#PWR013" H 8350 2600 50  0001 C CNN
 F 1 "+5V" H 8365 2923 50  0000 C CNN
 F 2 "" H 8350 2750 50  0001 C CNN
@@
 $EndComp
 $Comp
-L GND #PWR20
+L GND #PWR014
 U 1 1 592209F9
 P 9350 2850
-F 0 "#PWR20" H 9350 2600 50  0001 C CNN
+F 0 "#PWR014" H 9350 2600 50  0001 C CNN
 F 1 "GND" H 9355 2677 50  0000 C CNN
 F 2 "" H 9350 2850 50  0001 C CNN
@@
 $EndComp
 $Comp
-L GND #PWR14
+L GND #PWR015
 U 1 1 59220F59
 P 8000 5000
-F 0 "#PWR14" H 8000 4750 50  0001 C CNN
+F 0 "#PWR015" H 8000 4750 50  0001 C CNN
 F 1 "GND" H 8005 4827 50  0000 C CNN
 F 2 "" H 8000 5000 50  0001 C CNN
@@
 Connection ~ 8000 4800
 $Comp
-L +5V #PWR21
+L +5V #PWR016
 U 1 1 592212AC
 P 10000 3800
-F 0 "#PWR21" H 10000 3650 50  0001 C CNN
+F 0 "#PWR016" H 10000 3650 50  0001 C CNN
 F 1 "+5V" H 10015 3973 50  0000 C CNN
 F 2 "" H 10000 3800 50  0001 C CNN
@@
 $EndComp
 $Comp
-L +5V #PWR11
+L +5V #PWR017
 U 1 1 59223BEE
 P 6900 2650
-F 0 "#PWR11" H 6900 2500 50  0001 C CNN
+F 0 "#PWR017" H 6900 2500 50  0001 C CNN
 F 1 "+5V" H 6915 2823 50  0000 C CNN
 F 2 "" H 6900 2650 50  0001 C CNN
@@
 $EndComp
 $Comp
-L GND #PWR10
+L GND #PWR018
 U 1 1 592245AF
 P 6300 5450
-F 0 "#PWR10" H 6300 5200 50  0001 C CNN
+F 0 "#PWR018" H 6300 5200 50  0001 C CNN
 F 1 "GND" H 6305 5277 50  0000 C CNN
 F 2 "" H 6300 5450 50  0001 C CNN
@@
 Connection ~ 7700 3300
 $Comp
-L GND #PWR12
+L GND #PWR019
 U 1 1 59225578
 P 7300 3750
-F 0 "#PWR12" H 7300 3500 50  0001 C CNN
+F 0 "#PWR019" H 7300 3500 50  0001 C CNN
 F 1 "GND" H 7305 3577 50  0000 C CNN
 F 2 "" H 7300 3750 50  0001 C CNN
@@
 $EndComp
 $Comp
-L GND #PWR13
+L GND #PWR020
 U 1 1 592255B5
 P 7700 3750
-F 0 "#PWR13" H 7700 3500 50  0001 C CNN
+F 0 "#PWR020" H 7700 3500 50  0001 C CNN
 F 1 "GND" H 7705 3577 50  0000 C CNN
 F 2 "" H 7700 3750 50  0001 C CNN
@@
 $EndComp
 $Comp
-L PWR_FLAG #FLG2
+L PWR_FLAG #FLG021
 U 1 1 5922614D
 P 3250 3600
-F 0 "#FLG2" H 3250 3675 50  0001 C CNN
+F 0 "#FLG021" H 3250 3675 50  0001 C CNN
 F 1 "PWR_FLAG" H 3250 3774 50  0000 C CNN
 F 2 "" H 3250 3600 50  0001 C CNN
@@
 Connection ~ 3600 3700
 $Comp
-L PWR_FLAG #FLG1
+L PWR_FLAG #FLG022
 U 1 1 59226374
 P 2850 2750
-F 0 "#FLG1" H 2850 2825 50  0001 C CNN
+F 0 "#FLG022" H 2850 2825 50  0001 C CNN
 F 1 "PWR_FLAG" H 2850 2924 50  0000 C CNN
 F 2 "" H 2850 2750 50  0001 C CNN
@@
 Connection ~ 3200 2850
 $Comp
-L +5V #PWR6
+L +5V #PWR023
 U 1 1 59229303
 P 4650 2350
-F 0 "#PWR6" H 4650 2200 50  0001 C CNN
+F 0 "#PWR023" H 4650 2200 50  0001 C CNN
 F 1 "+5V" H 4665 2523 50  0000 C CNN
 F 2 "" H 4650 2350 50  0001 C CNN
@@
 F 0 "D3" V 7254 3679 50  0000 L CNN
 F 1 "3V6" V 7345 3679 50  0000 L CNN
-F 2 "" H 7300 3600 50  0001 C CNN
+F 2 "TO_SOT_Packages_SMD:SOT-23" H 7300 3600 50  0001 C CNN
 F 3 "" H 7300 3600 50  0001 C CNN
 	1    7300 3600
@@
 F 0 "D4" V 7654 3679 50  0000 L CNN
 F 1 "3V6" V 7745 3679 50  0000 L CNN
-F 2 "" H 7700 3600 50  0001 C CNN
+F 2 "TO_SOT_Packages_SMD:SOT-23" H 7700 3600 50  0001 C CNN
 F 3 "" H 7700 3600 50  0001 C CNN
 	1    7700 3600
